Commit message: Fix unit scale mismatch, correct transmission joint names, add wheel friction and cylinder collision geometry for Gazebo stability

File: urdf/mobile_robot.urdf (robot description, URDF)
Before this commit: robot mobile_robot, 6 links, 5 joints
Links:
- removed link base_link
- removed link left_front_link
- removed link left_rear_link
- removed link right_front_link
- removed link right_rear_link
- added link body1, mass 0.0314678; collision mesh filename=package://mobile_robot/meshes/Body1.stl scale=1 1 1; visual mesh filename=package://mobile_robot/meshes/Body1.stl scale=1 1 1
- added link front_left_wheel_1__body1, mass 0.003843; collision cylinder length=0.03 radius=0.065; visual mesh filename=package://mobile_robot/meshes/front_left_wheel_1__Body1.stl scale=1 1 1
- added link front_right_wheel_1__body1, mass 0.0039538; collision cylinder length=0.03 radius=0.065; visual mesh filename=package://mobile_robot/meshes/front_right_wheel_1__Body1.stl scale=1 1 1
- added link reae_right_wheel_1__body1, mass 0.00395256; collision mesh filename=package://mobile_robot/meshes/reae_right_wheel_1__Body1.stl scale=1 1 1; visual mesh filename=package://mobile_robot/meshes/reae_right_wheel_1__Body1.stl scale=1 1 1
- added link rear_left_wheel_1__body1, mass 0.00395314; collision mesh filename=package://mobile_robot/meshes/rear_left_wheel_1__Body1.stl scale=1 1 1; visual mesh filename=package://mobile_robot/meshes/rear_left_wheel_1__Body1.stl scale=1 1 1
Joints:
- removed joint left_front_joint
- removed joint left_rear_joint
- removed joint right_front_joint
- removed joint right_rear_joint
- added joint revolute_1: type continuous, parent body1, child front_left_wheel_1__body1, origin xyz=-0.225 0.17 0.045 rpy=0 -0 0, axis 1 0 0
- added joint revolute_2: type continuous, parent body1, child front_right_wheel_1__body1, origin xyz=0.225 0.17 0.045 rpy=0 -0 0, axis 1 0 0
- added joint revolute_3: type continuous, parent body1, child reae_right_wheel_1__body1, origin xyz=0.225 -0.17 0.045 rpy=0 -0 0, axis 1 0 0
- added joint revolute_4: type continuous, parent body1, child rear_left_wheel_1__body1, origin xyz=-0.225 -0.17 0.045 rpy=0 -0 0, axis 1 0 0
- joint fixed_node_to_root_joint: child base_link -> body1; origin xyz=0.00161778 0.0120001 0.00161092 rpy=0 -0 0 -> xyz=0.0631956 0.100605 -0.0138088 rpy=0 -0 0

Commit message: Working differential drive using libgazebo_ros_skid_steer_drive plugin

File: urdf/mobile_robot.urdf (robot description, URDF)
Before this commit: robot mobile_robot, 6 links, 5 joints
Links:
- link reae_right_wheel_1__body1: geometry collision cylinder length=0.03 radius=0.065; visual mesh filename=package://mobile_robot/meshes/reae_right_wheel_1__Body1.stl scale=1 1 1
- link rear_left_wheel_1__body1: geometry collision cylinder length=0.03 radius=0.065; visual mesh filename=package://mobile_robot/meshes/rear_left_wheel_1__Body1.stl scale=1 1 1
Joints:
- joint revolute_1: axis 1 0 0 -> -1 0 0
- joint revolute_2: axis 1 0 0 -> -1 0 0
- joint revolute_3: axis 1 0 0 -> -1 0 0
- joint revolute_4: axis 1 0 0 -> -1 0 0

Commit message: Add LiDAR sensor (link, joint, gazebo ray sensor plugin) and switch to turtlebot3_house world for testing

File: urdf/mobile_robot.urdf (robot description, URDF)
Before this commit: robot mobile_robot, 6 links, 5 joints
Links:
- added link lidar_link, mass 0.001; collision cylinder length=0.004 radius=0.0025; visual cylinder length=0.004 radius=0.0025
Joints:
- added joint lidar_joint: type fixed, parent body1, child lidar_link, origin xyz=0 -0.01 0.224 rpy=0 0 0

Commit message: Fix robot orientation mismatch: remove conflicting static root->body1 joint (leftover Onshape assembly-anchor artifact) that was creating two competing parents for body1 in the TF tree

File: urdf/mobile_robot.urdf (robot description, URDF)
Before this commit: robot mobile_robot, 7 links, 6 joints
Links:
- removed link root
Joints:
- removed joint fixed_node_to_root_joint

Commit message: Confirm working autonomous navigation; fix base_link frame convention and rosparam namespace nesting bug; update README

File: urdf/mobile_robot.urdf (robot description, URDF)
Before this commit: robot mobile_robot, 6 links, 5 joints
Links:
- added link base_link
Joints:
- added joint body1_to_base_link: type fixed, parent body1, child base_link, origin xyz=0 0 0 rpy=0 0 1.5708

Commit message: Add camera comparison screenshot and update README

File: urdf/mobile_robot.urdf (robot description, URDF)
Before this commit: robot mobile_robot, 7 links, 6 joints
Links:
- added link stereo_camera_link, mass 0.005; collision box size=0.02 0.08 0.02; visual box size=0.02 0.08 0.02
Joints:
- added joint stereo_camera_joint: type fixed, parent body1, child stereo_camera_link, origin xyz=0 0.25 0.158 rpy=0 0 1.5708
